File: ArchedArrayAZ100/slice_v6_zp.sch (EAGLE design)
At the start: 118 parts

Commit message: redid schematic for ArchedArray and modified LED part
Parts:
- removed U$1: TLC5955V0, ZacksLib:TLC5955V0
- added CHIP2: TLC5955V0, ZacksLib:TLC5955V0
Connections:
- new net N$294: D67.CATHODE, D76.CATHODE
- net GND: now also C2.1, C3.1, C4.1, C6.1, CHIP2.GND, CHIP2.GND2; no longer C2.2, C3.2, C4.2, C6.2, U$1.GND, U$1.GND2
- net GSCLK: now also CHIP2.GSCLK, U$3.GSCLK; no longer U$1.GSCLK, U$3.SCLK
- net LAT: now also CHIP2.LAT; no longer U$1.LAT
- net N$1: now also CHIP2.R0; no longer U$1.R0
- net N$10: now also CHIP2.B1; no longer U$1.B1
- net N$11: now also CHIP2.R7; no longer U$1.R7
- net N$12: now also CHIP2.G7; no longer U$1.G7
- net N$13: now also CHIP2.B7; no longer U$1.B7
- net N$14: now also CHIP2.R5; no longer U$1.R5
- net N$15: now also CHIP2.G5; no longer U$1.G5
- net N$16: now also CHIP2.B5; no longer U$1.B5
- net N$17: now also CHIP2.G6; no longer U$1.G6
- net N$18: now also CHIP2.B6; no longer U$1.B6
- net N$19: now also CHIP2.B4; no longer U$1.B4
- net N$2: now also CHIP2.R6; no longer U$1.R6
- net N$20: now also CHIP2.G4; no longer U$1.G4
- net N$21: now also CHIP2.R4; no longer U$1.R4
- net N$22: now also CHIP2.R3; no longer U$1.R3
- net N$23: now also CHIP2.G3; no longer U$1.G3
- net N$24: now also CHIP2.B3; no longer U$1.B3
- net N$25: now also CHIP2.G15; no longer U$1.G15
- net N$26: now also CHIP2.G11; no longer U$1.G11
- net N$27: now also CHIP2.R11; no longer U$1.R11
- net N$28: now also CHIP2.G8; no longer U$1.G8
- net N$287: now also CHIP2.SIN; no longer U$1.SIN
- net N$29: now also CHIP2.B8; no longer U$1.B8
- net N$291: now also CHIP2.SOUT; no longer U$1.SOUT
- net N$293: now also CHIP2.G0; no longer U$1.G0
- net N$3: now also CHIP2.B0; no longer U$1.B0
- net N$30: now also CHIP2.B15; no longer U$1.B15
- net N$31: now also CHIP2.R8; no longer U$1.R8
- net N$32: now also CHIP2.B9; no longer U$1.B9
- net N$33: now also CHIP2.G9; no longer U$1.G9
- net N$34: now also CHIP2.R14; no longer U$1.R14
- net N$35: now also CHIP2.R10; no longer U$1.R10
- net N$36: now also CHIP2.G12; no longer U$1.G12
- net N$37: now also CHIP2.B14; no longer U$1.B14
- net N$38: now also CHIP2.R9; no longer U$1.R9
- net N$39: now also CHIP2.R13; no longer U$1.R13
- net N$4: now also CHIP2.R2; no longer U$1.R2
- net N$40: now also CHIP2.G13; no longer U$1.G13
- net N$41: now also CHIP2.B13; no longer U$1.B13
- net N$42: now also CHIP2.G10; no longer U$1.G10
- net N$43: now also CHIP2.B10; no longer U$1.B10
- net N$44: now also CHIP2.B11; no longer U$1.B11
- net N$46: now also CHIP2.B12; no longer U$1.B12
- net N$47: now also CHIP2.R12; no longer U$1.R12
- net N$49: now also CHIP2.G14; no longer U$1.G14
- net N$5: now also CHIP2.G2; no longer U$1.G2
- net N$6: now also CHIP2.B2; no longer U$1.B2
- net N$7: now also CHIP2.R1; no longer U$1.R1
- net N$8: now also CHIP2.R15; no longer U$1.R15
- net N$9: now also CHIP2.G1; no longer U$1.G1
- net SCLK: now also CHIP2.SCLK, U$3.SCLK; no longer U$1.SCLK, U$3.GSCLK
- net VCC: now also C2.2, C3.2, C4.2, C6.2, CHIP2.VCC; no longer C2.1, C3.1, C4.1, C6.1, D67.CATHODE, D76.CATHODE, U$1.VCC
Other:
- moved on the sheet: C1, C2, C3, C4, C5, C6, D1, D10, D11, D12, D13, D14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

Commit message: Finished TLC5955 initial board
Parts:
- renumbered CHIP2 to CHIP_2, U$2 to CHIP_6, U$3 to CHIP_5, U$4 to CHIP_1, U$5 to CHIP_3, U$6 to CHIP_4
Connections:
- net DATA_OUT: now also SOUT2.1; no longer SOUT6.1
- net N$1: now also CHIP_6.R0; no longer CHIP_2.R0
- net N$10: now also CHIP_6.B1; no longer CHIP_2.B1
- net N$11: now also CHIP_6.R7; no longer CHIP_2.R7
- net N$12: now also CHIP_6.G7; no longer CHIP_2.G7
- net N$13: now also CHIP_6.B7; no longer CHIP_2.B7
- net N$14: now also CHIP_6.R5; no longer CHIP_2.R5
- net N$15: now also CHIP_6.G5; no longer CHIP_2.G5
- net N$16: now also CHIP_6.B5; no longer CHIP_2.B5
- net N$17: now also CHIP_6.G6; no longer CHIP_2.G6
- net N$18: now also CHIP_6.B6; no longer CHIP_2.B6
- net N$189: now also CHIP_2.R0; no longer CHIP_3.R0
- net N$19: now also CHIP_6.B4; no longer CHIP_2.B4
- net N$190: now also CHIP_2.B0; no longer CHIP_3.B0
- net N$191: now also CHIP_2.R2; no longer CHIP_3.R2
- net N$192: now also CHIP_2.G2; no longer CHIP_3.G2
- net N$193: now also CHIP_2.B2; no longer CHIP_3.B2
- net N$194: now also CHIP_2.R1; no longer CHIP_3.R1
- net N$195: now also CHIP_2.G1; no longer CHIP_3.G1
- net N$196: now also CHIP_2.B1; no longer CHIP_3.B1
- net N$197: now also CHIP_2.R7; no longer CHIP_3.R7
- net N$198: now also CHIP_2.G7; no longer CHIP_3.G7
- net N$199: now also CHIP_2.B7; no longer CHIP_3.B7
- net N$2: now also CHIP_6.R6; no longer CHIP_2.R6
- net N$20: now also CHIP_6.G4; no longer CHIP_2.G4
- net N$200: now also CHIP_2.R5; no longer CHIP_3.R5
- net N$201: now also CHIP_2.G5; no longer CHIP_3.G5
- net N$202: now also CHIP_2.B5; no longer CHIP_3.B5
- net N$203: now also CHIP_2.R6; no longer CHIP_3.R6
- net N$204: now also CHIP_2.G6; no longer CHIP_3.G6
- net N$205: now also CHIP_2.B6; no longer CHIP_3.B6
- net N$206: now also CHIP_2.B4; no longer CHIP_3.B4
- net N$207: now also CHIP_2.G4; no longer CHIP_3.G4
- net N$208: now also CHIP_2.R4; no longer CHIP_3.R4
- net N$209: now also CHIP_2.R3; no longer CHIP_3.R3
- net N$21: now also CHIP_6.R4; no longer CHIP_2.R4
- net N$210: now also CHIP_2.G3; no longer CHIP_3.G3
- net N$211: now also CHIP_2.B3; no longer CHIP_3.B3
- net N$212: now also CHIP_2.B8; no longer CHIP_3.B8
- net N$213: now also CHIP_2.R8; no longer CHIP_3.R8
- net N$214: now also CHIP_2.B9; no longer CHIP_3.B9
- net N$215: now also CHIP_2.G9; no longer CHIP_3.G9
- net N$216: now also CHIP_2.R10; no longer CHIP_3.R10
- net N$217: now also CHIP_2.G11; no longer CHIP_3.G11
- net N$218: now also CHIP_2.R11; no longer CHIP_3.R11
- net N$219: now also CHIP_2.G8; no longer CHIP_3.G8
- net N$22: now also CHIP_6.R3; no longer CHIP_2.R3
- net N$220: now also CHIP_2.R9; no longer CHIP_3.R9
- net N$221: now also CHIP_2.G10; no longer CHIP_3.G10
- net N$222: now also CHIP_2.B10; no longer CHIP_3.B10
- net N$223: now also CHIP_2.B11; no longer CHIP_3.B11
- net N$224: now also CHIP_2.R15; no longer CHIP_3.R15
- net N$225: now also CHIP_2.G15; no longer CHIP_3.G15
- net N$226: now also CHIP_2.B15; no longer CHIP_3.B15
- net N$227: now also CHIP_2.R14; no longer CHIP_3.R14
- net N$228: now also CHIP_2.B14; no longer CHIP_3.B14
- net N$229: now also CHIP_2.R13; no longer CHIP_3.R13
- net N$23: now also CHIP_6.G3; no longer CHIP_2.G3
- net N$230: now also CHIP_2.G13; no longer CHIP_3.G13
- net N$231: now also CHIP_2.B13; no longer CHIP_3.B13
- net N$232: now also CHIP_2.B12; no longer CHIP_3.B12
- net N$233: now also CHIP_2.R12; no longer CHIP_3.R12
- net N$234: now also CHIP_2.G14; no longer CHIP_3.G14
- net N$235: now also CHIP_2.G12; no longer CHIP_3.G12
- net N$236: now also CHIP_3.R0; no longer CHIP_4.R0
- net N$237: now also CHIP_3.B0; no longer CHIP_4.B0
- net N$238: now also CHIP_3.R2; no longer CHIP_4.R2
- net N$239: now also CHIP_3.G2; no longer CHIP_4.G2
- net N$24: now also CHIP_6.B3; no longer CHIP_2.B3
- net N$240: now also CHIP_3.B2; no longer CHIP_4.B2
- net N$241: now also CHIP_3.R1; no longer CHIP_4.R1
- net N$242: now also CHIP_3.G1; no longer CHIP_4.G1
- net N$243: now also CHIP_3.B1; no longer CHIP_4.B1
- net N$244: now also CHIP_3.R7; no longer CHIP_4.R7
- net N$245: now also CHIP_3.G7; no longer CHIP_4.G7
- net N$246: now also CHIP_3.B7; no longer CHIP_4.B7
- net N$247: now also CHIP_3.R5; no longer CHIP_4.R5
- net N$248: now also CHIP_3.G5; no longer CHIP_4.G5
- net N$249: now also CHIP_3.B5; no longer CHIP_4.B5
- net N$25: now also CHIP_6.G15; no longer CHIP_2.G15
- net N$250: now also CHIP_3.R6; no longer CHIP_4.R6
- net N$251: now also CHIP_3.G6; no longer CHIP_4.G6
- net N$252: now also CHIP_3.B6; no longer CHIP_4.B6
- net N$253: now also CHIP_3.B4; no longer CHIP_4.B4
- net N$254: now also CHIP_3.G4; no longer CHIP_4.G4
- net N$255: now also CHIP_3.R4; no longer CHIP_4.R4
- net N$256: now also CHIP_3.R3; no longer CHIP_4.R3
- net N$257: now also CHIP_3.G3; no longer CHIP_4.G3
- net N$258: now also CHIP_3.B3; no longer CHIP_4.B3
- net N$259: now also CHIP_3.B8; no longer CHIP_4.B8
- net N$26: now also CHIP_6.G11; no longer CHIP_2.G11
- net N$260: now also CHIP_3.R8; no longer CHIP_4.R8
- net N$261: now also CHIP_3.B9; no longer CHIP_4.B9
- net N$262: now also CHIP_3.G9; no longer CHIP_4.G9
- net N$263: now also CHIP_3.R10; no longer CHIP_4.R10
- net N$264: now also CHIP_3.G11; no longer CHIP_4.G11
- net N$265: now also CHIP_3.R11; no longer CHIP_4.R11
- net N$266: now also CHIP_3.G8; no longer CHIP_4.G8
- net N$267: now also CHIP_3.R9; no longer CHIP_4.R9
- net N$268: now also CHIP_3.G10; no longer CHIP_4.G10
- net N$269: now also CHIP_3.B10; no longer CHIP_4.B10
- net N$27: now also CHIP_6.R11; no longer CHIP_2.R11
- net N$270: now also CHIP_3.B11; no longer CHIP_4.B11
- net N$271: now also CHIP_3.R15; no longer CHIP_4.R15
- net N$272: now also CHIP_3.G15; no longer CHIP_4.G15
- net N$273: now also CHIP_3.B15; no longer CHIP_4.B15
- net N$274: now also CHIP_3.R14; no longer CHIP_4.R14
- net N$275: now also CHIP_3.B14; no longer CHIP_4.B14
- net N$276: now also CHIP_3.R13; no longer CHIP_4.R13
- net N$277: now also CHIP_3.G13; no longer CHIP_4.G13
- net N$278: now also CHIP_3.B13; no longer CHIP_4.B13
- net N$279: now also CHIP_3.B12; no longer CHIP_4.B12
- net N$28: now also CHIP_6.G8; no longer CHIP_2.G8
- net N$280: now also CHIP_3.R12; no longer CHIP_4.R12
- net N$281: now also CHIP_3.G14; no longer CHIP_4.G14
- net N$282: now also CHIP_3.G12; no longer CHIP_4.G12
- net N$283: now also SOUT4.1; no longer SOUT3.1
- net N$286: now also SOUT6.1; no longer SOUT4.1
- net N$288: now also CHIP_3.G0; no longer CHIP_4.G0
- net N$29: now also CHIP_6.B8; no longer CHIP_2.B8
- net N$290: now also CHIP_4.G0; no longer CHIP_6.G0
- net N$291: now also SOUT3.1; no longer SOUT2.1
- net N$293: now also CHIP_6.G0; no longer CHIP_2.G0
- net N$298: now also CHIP_2.G0; no longer CHIP_3.G0
- net N$3: now also CHIP_6.B0; no longer CHIP_2.B0
- net N$30: now also CHIP_6.B15; no longer CHIP_2.B15
- net N$31: now also CHIP_6.R8; no longer CHIP_2.R8
- net N$32: now also CHIP_6.B9; no longer CHIP_2.B9
- net N$33: now also CHIP_6.G9; no longer CHIP_2.G9
- net N$34: now also CHIP_6.R14; no longer CHIP_2.R14
- net N$35: now also CHIP_6.R10; no longer CHIP_2.R10
- net N$36: now also CHIP_6.G12; no longer CHIP_2.G12
- net N$37: now also CHIP_6.B14; no longer CHIP_2.B14
- net N$38: now also CHIP_6.R9; no longer CHIP_2.R9
- net N$39: now also CHIP_6.R13; no longer CHIP_2.R13
- net N$4: now also CHIP_6.R2; no longer CHIP_2.R2
- net N$40: now also CHIP_6.G13; no longer CHIP_2.G13
- net N$41: now also CHIP_6.B13; no longer CHIP_2.B13
- net N$42: now also CHIP_6.G10; no longer CHIP_2.G10
- net N$43: now also CHIP_6.B10; no longer CHIP_2.B10
- net N$44: now also CHIP_6.B11; no longer CHIP_2.B11
- net N$45: now also CHIP_4.R0; no longer CHIP_6.R0
- net N$46: now also CHIP_6.B12; no longer CHIP_2.B12
- net N$47: now also CHIP_6.R12; no longer CHIP_2.R12
- net N$48: now also CHIP_4.B0; no longer CHIP_6.B0
- net N$49: now also CHIP_6.G14; no longer CHIP_2.G14
- net N$5: now also CHIP_6.G2; no longer CHIP_2.G2
- net N$50: now also CHIP_4.R2; no longer CHIP_6.R2
- net N$51: now also CHIP_4.G2; no longer CHIP_6.G2
- net N$52: now also CHIP_4.B2; no longer CHIP_6.B2
- net N$53: now also CHIP_4.R1; no longer CHIP_6.R1
- net N$54: now also CHIP_4.G1; no longer CHIP_6.G1
- net N$55: now also CHIP_4.B1; no longer CHIP_6.B1
- net N$56: now also CHIP_4.R7; no longer CHIP_6.R7
- net N$57: now also CHIP_4.G7; no longer CHIP_6.G7
- net N$58: now also CHIP_4.B7; no longer CHIP_6.B7
- net N$59: now also CHIP_4.R5; no longer CHIP_6.R5
- net N$6: now also CHIP_6.B2; no longer CHIP_2.B2
- net N$60: now also CHIP_4.G5; no longer CHIP_6.G5
- net N$61: now also CHIP_4.B5; no longer CHIP_6.B5
- net N$62: now also CHIP_4.R6; no longer CHIP_6.R6
- net N$63: now also CHIP_4.G6; no longer CHIP_6.G6
- net N$64: now also CHIP_4.B6; no longer CHIP_6.B6
- net N$65: now also CHIP_4.B4; no longer CHIP_6.B4
- net N$66: now also CHIP_4.G4; no longer CHIP_6.G4
- net N$67: now also CHIP_4.R4; no longer CHIP_6.R4
- net N$68: now also CHIP_4.R3; no longer CHIP_6.R3
- net N$69: now also CHIP_4.G3; no longer CHIP_6.G3
- net N$7: now also CHIP_6.R1; no longer CHIP_2.R1
- net N$70: now also CHIP_4.B3; no longer CHIP_6.B3
- net N$71: now also CHIP_4.B8; no longer CHIP_6.B8
- net N$72: now also CHIP_4.R8; no longer CHIP_6.R8
- net N$73: now also CHIP_4.B9; no longer CHIP_6.B9
- net N$74: now also CHIP_4.G9; no longer CHIP_6.G9
- net N$75: now also CHIP_4.R10; no longer CHIP_6.R10
- net N$76: now also CHIP_4.G11; no longer CHIP_6.G11
- net N$77: now also CHIP_4.R11; no longer CHIP_6.R11
- net N$78: now also CHIP_4.G8; no longer CHIP_6.G8
- net N$79: now also CHIP_4.R9; no longer CHIP_6.R9
- net N$8: now also CHIP_6.R15; no longer CHIP_2.R15
- net N$80: now also CHIP_4.G10; no longer CHIP_6.G10
- net N$81: now also CHIP_4.B10; no longer CHIP_6.B10
- net N$82: now also CHIP_4.B11; no longer CHIP_6.B11
- net N$83: now also CHIP_4.R15; no longer CHIP_6.R15
- net N$84: now also CHIP_4.G15; no longer CHIP_6.G15
- net N$85: now also CHIP_4.B15; no longer CHIP_6.B15
- net N$86: now also CHIP_4.R14; no longer CHIP_6.R14
- net N$87: now also CHIP_4.B14; no longer CHIP_6.B14
- net N$88: now also CHIP_4.R13; no longer CHIP_6.R13
- net N$89: now also CHIP_4.G13; no longer CHIP_6.G13
- net N$9: now also CHIP_6.G1; no longer CHIP_2.G1
- net N$90: now also CHIP_4.B13; no longer CHIP_6.B13
- net N$91: now also CHIP_4.B12; no longer CHIP_6.B12
- net N$92: now also CHIP_4.R12; no longer CHIP_6.R12
- net N$93: now also CHIP_4.G14; no longer CHIP_6.G14
- net N$94: now also CHIP_4.G12; no longer CHIP_6.G12
Other:
- moved on the sheet: C1, C2, C5, C6, D1, D10, D11, D12, D13, D14, D15, D16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
