File: PlanarArrayCellScope/ArrayC_v0zp.sch (EAGLE design)
At the start: 121 parts

Commit message: Updated Planar Array Designs
Parts:
- removed LED100, LED101, LED102, LED103, LED104, LED105, LED106, LED107, LED108, LED109, LED110, LED111, LED112, LED113, LED114, LED115, LED116, LED117, LED118, LED119, LED120, LED81, LED82, LED83, LED84, LED85, LED86, LED87, LED88, LED89, LED90, LED91, LED92, LED93, LED94, LED95, LED96, LED97, LED98, LED99: KB_APTF1616V0, ZacksLib:KB_APTF1616V0
- LED00, LED01, LED02, LED03, LED04, LED05, LED06, LED07, LED08, LED09, LED10, LED11, LED12, LED13, LED14, LED15, LED16, LED17, LED18, LED19, LED20, LED21, LED22, LED23, LED24, LED25, LED26, LED27, LED28, LED29, LED30, LED31, LED32, LED33, LED34, LED35, LED36, LED37, LED38, LED39, LED40, LED41, LED42, LED43, LED44, LED45, LED46, LED47, LED48, LED49, LED50, LED51, LED52, LED53, LED54, LED55, LED56, LED57, LED58, LED59, LED60, LED61, LED62, LED63, LED64, LED65, LED66, LED67, LED68, LED69, LED70, LED71, LED72, LED73, LED74, LED75, LED76, LED77, LED78, LED79, LED80: device ZacksLib:KB_APTF1616V0 -> WallerLabLib:KB_APTF1616V0
