File: PlanarArrayCellScope/ArrayC_v2zp.brd (EAGLE design)
At the start: 41.1 x 41.1 mm, 131 parts

Commit message: Updated Planar Array Designs
Parts:
- removed LED00, LED01, LED02, LED03, LED04, LED05, LED06, LED07, LED08, LED09, LED10, LED100, LED101, LED102, LED103, LED104, LED105, LED106, LED107, LED108, LED109, LED11, LED110, LED111, LED112, LED113, LED114, LED115, LED116, LED117, LED118, LED119, LED12, LED120, LED13, LED14, LED15, LED16, LED17, LED18, LED19, LED20, LED21, LED22, LED23, LED24, LED25, LED26, LED27, LED28, LED29, LED30, LED31, LED32, LED33, LED34, LED35, LED36, LED37, LED38, LED39, LED40, LED41, LED42, LED43, LED44, LED45, LED46, LED47, LED48, LED49, LED50, LED51, LED52, LED53, LED54, LED55, LED56, LED57, LED58, LED59, LED60, LED61, LED62, LED63, LED64, LED65, LED66, LED67, LED68, LED69, LED70, LED71, LED72, LED73, LED74, LED75, LED76, LED77, LED78, LED79, LED80, LED81, LED82, LED83, LED84, LED85, LED86, LED87, LED88, LED89, LED90, LED91, LED92, LED93, LED94, LED95, LED96, LED97, LED98, LED99: KB_APTF1616V0, ZacksLib:KB_RGBLED_APTF1616
- moved U$3 43.1 mm to (61.9, 18.6)
- moved U$2 32.3 mm to (56.8, 5.50)
- moved U$6 29.0 mm to (61.5, 41.6)
- moved U$8 27.4 mm to (24.8, 38.0)
- moved U$4 12.0 mm to (37.5, 37.5), turned to 90 degrees
- moved U$5 5.43 mm to (16.2, 54.5)
Connections:
- removed net N$367: LED40.P1, LED41.P1, LED42.P1, LED43.P1, LED44.P1, LED45.P1, LED46.P1, LED47.P1, LED80.P1, LED81.P1, LED82.P1, LED83.P1, LED84.P1, LED86.P1, LED87.P1
- removed net N$369: LED00.P1, LED01.P1, LED02.P1, LED03.P1, LED04.P1, LED05.P1, LED06.P1, LED07.P1
- removed net N$374: LED24.P1, LED25.P1, LED26.P1, LED27.P1, LED28.P1, LED29.P1, LED30.P1, LED31.P1, LED48.P1, LED49.P1, LED50.P1, LED51.P1, LED52.P1, LED53.P1, LED54.P1, LED55.P1
- removed net N$384: LED56.P1, LED57.P1, LED58.P1, LED59.P1, LED60.P1, LED61.P1, LED62.P1, LED63.P1, LED64.P1, LED65.P1, LED66.P1, LED67.P1, LED68.P1, LED69.P1, LED70.P1, LED71.P1
- net 3.3V: no longer LED08.P1, LED09.P1, LED10.P1, LED100.P1, LED101.P1, LED102.P1, LED103.P1, LED104.P1, LED105.P1, LED106.P1, LED107.P1, LED108.P1, LED109.P1, LED11.P1, LED110.P1, LED111.P1, LED112.P1, LED113.P1, LED114.P1, LED115.P1, LED116.P1, LED117.P1, LED118.P1, LED119.P1, LED12.P1, LED120.P1, LED13.P1, LED14.P1, LED15.P1, LED16.P1, LED17.P1, LED18.P1, LED19.P1, LED20.P1, LED21.P1, LED22.P1, LED23.P1, LED32.P1, LED33.P1, LED34.P1, LED35.P1, LED36.P1, LED37.P1, LED38.P1, LED39.P1, LED72.P1, LED73.P1, LED74.P1, LED75.P1, LED76.P1, LED77.P1, LED78.P1, LED79.P1, LED88.P1, LED89.P1, LED90.P1, LED91.P1, LED92.P1, LED93.P1, LED94.P1, LED95.P1, LED96.P1, LED97.P1, LED98.P1, LED99.P1
- net N$1: no longer LED00.P2
- net N$10: no longer LED03.P2
- net N$100: no longer LED17.P4
- net N$101: no longer LED18.P2
- net N$102: no longer LED18.P3
- net N$103: no longer LED18.P4
- net N$104: no longer LED19.P2
- net N$105: no longer LED19.P3
- net N$106: no longer LED19.P4
- net N$107: no longer LED20.P2
- net N$108: no longer LED20.P3
- net N$109: no longer LED20.P4
- net N$11: no longer LED03.P3
- net N$110: no longer LED21.P2
- net N$111: no longer LED21.P3
- net N$112: no longer LED21.P4
- net N$113: no longer LED22.P2
- net N$114: no longer LED22.P3
- net N$115: no longer LED22.P4
- net N$116: no longer LED23.P2
- net N$117: no longer LED23.P3
- net N$118: no longer LED23.P4
- net N$119: no longer LED24.P4
- net N$12: no longer LED03.P4
- net N$120: no longer LED24.P3
- net N$121: no longer LED24.P2
- net N$122: no longer LED25.P4
- net N$123: no longer LED25.P3
- net N$124: no longer LED25.P2
- net N$125: no longer LED26.P4
- net N$126: no longer LED26.P3
- net N$127: no longer LED26.P2
- net N$128: no longer LED27.P4
- net N$129: no longer LED27.P3
- net N$13: no longer LED04.P2
- net N$130: no longer LED28.P4
- net N$131: no longer LED28.P3
- net N$132: no longer LED28.P2
- net N$133: no longer LED29.P4
- net N$134: no longer LED29.P3
- net N$135: no longer LED29.P2
- net N$136: no longer LED30.P4
- net N$137: no longer LED30.P3
- net N$138: no longer LED30.P2
- net N$139: no longer LED31.P4
- net N$14: no longer LED04.P3
- net N$140: no longer LED31.P3
- net N$141: no longer LED31.P2
- net N$142: no longer LED64.P2
- net N$143: no longer LED48.P2
- net N$144: no longer LED48.P3
- net N$145: no longer LED48.P4
- net N$146: no longer LED49.P2
- net N$147: no longer LED49.P3
- net N$148: no longer LED49.P4
- net N$149: no longer LED50.P2
- net N$15: no longer LED04.P4
- net N$150: no longer LED50.P3
- net N$151: no longer LED50.P4
- net N$152: no longer LED51.P2
- net N$153: no longer LED51.P3
- net N$154: no longer LED51.P4
- net N$155: no longer LED52.P2
- net N$156: no longer LED52.P3
- net N$157: no longer LED52.P4
- net N$158: no longer LED53.P2
- net N$159: no longer LED53.P3
- net N$16: no longer LED05.P2
- net N$160: no longer LED53.P4
- net N$161: no longer LED54.P2
- net N$162: no longer LED54.P3
- net N$163: no longer LED54.P4
- net N$164: no longer LED55.P2
- net N$165: no longer LED55.P3
- net N$166: no longer LED55.P4
- net N$167: no longer LED56.P4
- net N$168: no longer LED56.P3
- net N$169: no longer LED56.P2
- net N$17: no longer LED05.P3
- net N$170: no longer LED57.P4
- net N$171: no longer LED57.P3
- net N$172: no longer LED57.P2
- net N$173: no longer LED58.P4
- net N$174: no longer LED58.P3
- net N$175: no longer LED58.P2
- net N$176: no longer LED59.P4
- net N$177: no longer LED59.P3
- net N$178: no longer LED60.P4
- net N$179: no longer LED60.P3
- net N$18: no longer LED05.P4
- net N$180: no longer LED60.P2
- net N$181: no longer LED61.P4
- net N$182: no longer LED61.P3
- net N$183: no longer LED61.P2
- net N$184: no longer LED62.P4
- net N$185: no longer LED62.P3
- net N$186: no longer LED62.P2
- net N$187: no longer LED63.P4
- net N$188: no longer LED63.P3
- net N$189: no longer LED63.P2
- net N$19: no longer LED06.P2
- net N$190: no longer LED64.P3
- net N$191: no longer LED64.P4
- net N$192: no longer LED65.P2
- net N$193: no longer LED65.P3
- net N$194: no longer LED65.P4
- net N$195: no longer LED66.P2
- net N$196: no longer LED66.P3
- net N$197: no longer LED66.P4
- net N$198: no longer LED67.P2
- net N$199: no longer LED67.P3
- net N$2: no longer LED00.P3
- net N$20: no longer LED06.P3
- net N$200: no longer LED67.P4
- net N$201: no longer LED68.P2
- net N$202: no longer LED68.P3
- net N$203: no longer LED68.P4
- net N$204: no longer LED69.P2
- net N$205: no longer LED69.P3
- net N$206: no longer LED69.P4
- net N$207: no longer LED70.P2
- net N$208: no longer LED70.P3
- net N$209: no longer LED70.P4
- net N$21: no longer LED06.P4
- net N$210: no longer LED71.P2
- net N$211: no longer LED71.P3
- net N$212: no longer LED71.P4
- net N$213: no longer LED72.P4
- net N$214: no longer LED72.P3
- net N$215: no longer LED72.P2
- net N$216: no longer LED73.P4
- net N$217: no longer LED73.P3
- net N$218: no longer LED73.P2
- net N$219: no longer LED74.P4
- net N$22: no longer LED07.P2
- net N$220: no longer LED74.P3
- net N$221: no longer LED74.P2
- net N$222: no longer LED75.P4
- net N$223: no longer LED75.P3
- net N$224: no longer LED76.P4
- net N$225: no longer LED76.P3
- net N$226: no longer LED76.P2
- net N$227: no longer LED77.P4
- net N$228: no longer LED77.P3
- net N$229: no longer LED77.P2
- net N$23: no longer LED07.P3
- net N$230: no longer LED78.P4
- net N$231: no longer LED78.P3
- net N$232: no longer LED78.P2
- net N$233: no longer LED79.P4
- net N$234: no longer LED79.P3
- net N$235: no longer LED79.P2
- net N$236: no longer LED80.P2
- net N$237: no longer LED80.P3
- net N$238: no longer LED80.P4
- net N$239: no longer LED81.P2
- net N$24: no longer LED07.P4
- net N$240: no longer LED81.P3
- net N$241: no longer LED81.P4
- net N$242: no longer LED82.P2
- net N$243: no longer LED82.P3
- net N$244: no longer LED82.P4
- net N$245: no longer LED83.P2
- net N$246: no longer LED83.P3
- net N$247: no longer LED83.P4
- net N$248: no longer LED84.P2
- net N$249: no longer LED84.P3
- net N$25: no longer LED08.P4
- net N$250: no longer LED84.P4
- net N$251: no longer LED85.P2
- net N$252: no longer LED85.P3
- net N$253: no longer LED85.P4
- net N$254: no longer LED86.P2
- net N$255: no longer LED86.P3
- net N$256: no longer LED86.P4
- net N$257: no longer LED87.P2
- net N$258: no longer LED87.P3
- net N$259: no longer LED87.P4
- net N$26: no longer LED08.P3
- net N$260: no longer LED88.P4
- net N$261: no longer LED88.P3
- net N$262: no longer LED88.P2
- net N$263: no longer LED89.P4
- net N$264: no longer LED89.P3
- net N$265: no longer LED89.P2
- net N$266: no longer LED90.P4
- net N$267: no longer LED90.P3
- net N$268: no longer LED90.P2
- net N$269: no longer LED91.P4
- net N$27: no longer LED08.P2
- net N$270: no longer LED91.P3
- net N$271: no longer LED92.P4
- net N$272: no longer LED92.P3
- net N$273: no longer LED92.P2
- net N$274: no longer LED93.P4
- net N$275: no longer LED93.P3
- net N$276: no longer LED93.P2
- net N$277: no longer LED94.P4
- net N$278: no longer LED94.P3
- net N$279: no longer LED94.P2
- net N$28: no longer LED09.P4
- net N$280: no longer LED95.P4
- net N$281: no longer LED95.P3
- net N$282: no longer LED95.P2
- net N$283: no longer LED96.P2
- net N$284: no longer LED96.P3
- net N$285: no longer LED96.P4
- net N$286: no longer LED97.P2
- net N$287: no longer LED97.P3
- net N$288: no longer LED97.P4
- net N$289: no longer LED98.P2
- net N$29: no longer LED09.P3
- net N$290: no longer LED98.P3
- net N$291: no longer LED98.P4
- net N$292: no longer LED99.P2
- net N$293: no longer LED99.P3
- net N$294: no longer LED99.P4
- net N$295: no longer LED100.P2
- net N$296: no longer LED100.P3
- net N$297: no longer LED100.P4
- net N$298: no longer LED101.P2
- net N$299: no longer LED101.P3
- net N$3: no longer LED00.P4
- net N$30: no longer LED09.P2
- net N$300: no longer LED101.P4
- net N$301: no longer LED102.P2
- net N$302: no longer LED102.P3
- net N$303: no longer LED102.P4
- net N$304: no longer LED103.P2
- net N$305: no longer LED103.P3
- net N$306: no longer LED103.P4
- net N$307: no longer LED104.P4
- net N$308: no longer LED104.P3
- net N$309: no longer LED104.P2
- net N$31: no longer LED10.P4
- net N$310: no longer LED105.P4
- net N$311: no longer LED105.P3
- net N$312: no longer LED105.P2
- net N$313: no longer LED106.P4
- net N$314: no longer LED106.P3
- net N$315: no longer LED106.P2
- net N$316: no longer LED107.P4
- net N$317: no longer LED107.P3
- net N$318: no longer LED108.P4
- net N$319: no longer LED108.P3
- net N$32: no longer LED10.P3
- net N$320: no longer LED108.P2
- net N$321: no longer LED109.P4
- net N$322: no longer LED109.P3
- net N$323: no longer LED109.P2
- net N$324: no longer LED110.P4
- net N$325: no longer LED110.P3
- net N$326: no longer LED110.P2
- net N$327: no longer LED111.P4
- net N$328: no longer LED111.P3
- net N$329: no longer LED111.P2
- net N$33: no longer LED10.P2
- net N$330: no longer LED112.P2
- net N$331: no longer LED112.P3
- net N$332: no longer LED112.P4
- net N$333: no longer LED113.P2
- net N$334: no longer LED113.P3
- net N$335: no longer LED113.P4
- net N$336: no longer LED114.P2
- net N$337: no longer LED114.P3
- net N$338: no longer LED114.P4
- net N$339: no longer LED115.P2
- net N$34: no longer LED11.P4
- net N$340: no longer LED115.P3
- net N$341: no longer LED115.P4
- net N$342: no longer LED116.P2
- net N$343: no longer LED116.P3
- net N$344: no longer LED116.P4
- net N$345: no longer LED117.P2
- net N$346: no longer LED117.P3
- net N$347: no longer LED117.P4
- net N$348: no longer LED118.P2
- net N$349: no longer LED118.P3
- net N$35: no longer LED11.P3
- net N$350: no longer LED118.P4
- net N$351: no longer LED119.P2
- net N$352: no longer LED119.P3
- net N$353: no longer LED119.P4
- net N$354: no longer LED120.P4
- net N$355: no longer LED120.P3
- net N$356: no longer LED120.P2
- net N$36: no longer LED12.P4
- net N$364: no longer LED107.P2
- net N$368: no longer LED43.P2
- net N$37: no longer LED12.P3
- net N$370: no longer LED11.P2
- net N$371: no longer LED91.P2
- net N$372: no longer LED75.P2
- net N$373: no longer LED59.P2
- net N$375: no longer LED27.P2
- net N$38: no longer LED12.P2
- net N$39: no longer LED13.P4
- net N$4: no longer LED01.P2
- net N$40: no longer LED13.P3
- net N$41: no longer LED13.P2
- net N$42: no longer LED14.P4
- net N$43: no longer LED14.P3
- net N$44: no longer LED14.P2
- net N$45: no longer LED15.P4
- net N$46: no longer LED15.P3
- net N$47: no longer LED15.P2
- net N$48: no longer LED32.P2
- net N$49: no longer LED32.P3
- net N$5: no longer LED01.P3
- net N$50: no longer LED32.P4
- net N$51: no longer LED33.P2
- net N$52: no longer LED33.P3
- net N$53: no longer LED33.P4
- net N$54: no longer LED34.P2
- net N$55: no longer LED34.P3
- net N$56: no longer LED34.P4
- net N$57: no longer LED35.P2
- net N$58: no longer LED35.P3
- net N$59: no longer LED35.P4
- net N$6: no longer LED01.P4
- net N$60: no longer LED36.P2
- net N$61: no longer LED36.P3
- net N$62: no longer LED36.P4
- net N$63: no longer LED37.P2
- net N$64: no longer LED37.P3
- net N$65: no longer LED37.P4
- net N$66: no longer LED38.P2
- net N$67: no longer LED38.P3
- net N$68: no longer LED38.P4
- net N$69: no longer LED39.P2
- net N$7: no longer LED02.P2
- net N$70: no longer LED39.P3
- net N$71: no longer LED39.P4
- net N$72: no longer LED40.P4
- net N$73: no longer LED40.P3
- net N$74: no longer LED40.P2
- net N$75: no longer LED41.P4
- net N$76: no longer LED41.P3
- net N$77: no longer LED41.P2
- net N$78: no longer LED42.P4
- net N$79: no longer LED42.P3
- net N$8: no longer LED02.P3
- net N$80: no longer LED42.P2
- net N$81: no longer LED43.P4
- net N$82: no longer LED43.P3
- net N$83: no longer LED44.P4
- net N$84: no longer LED44.P3
- net N$85: no longer LED44.P2
- net N$86: no longer LED45.P4
- net N$87: no longer LED45.P3
- net N$88: no longer LED45.P2
- net N$89: no longer LED46.P4
- net N$9: no longer LED02.P4
- net N$90: no longer LED46.P3
- net N$91: no longer LED46.P2
- net N$92: no longer LED47.P4
- net N$93: no longer LED47.P3
- net N$94: no longer LED47.P2
- net N$95: no longer LED16.P2
- net N$96: no longer LED16.P3
- net N$97: no longer LED16.P4
- net N$98: no longer LED17.P2
- net N$99: no longer LED17.P3
Routing:
- net N$361: track 0.00 -> 5.71 mm
- net N$106: track 4.03 -> 0.00 mm, vias 1 -> 0
Other:
- board size 41.1 x 41.1 mm -> 64.4 x 64.4 mm
