File: PlanarArrayCellScope/ArrayF_v0zp.brd (EAGLE design)
At the start: 80 x 34.6 mm, 111 parts

Commit message: Updated Planar Array Designs
Parts:
- added LED111, LED112, LED113, LED114, LED115, LED116, LED117, LED118, LED119, LED120, LED121, LED122, LED123, LED124, LED125, LED126, LED127, LED128, LED129, LED130, LED131, LED132, LED133, LED134, LED135, LED136, LED137, LED138, LED139, LED140, LED141, LED142, LED143, LED144, LED145, LED146, LED147, LED148, LED149, LED150, LED151, LED152, LED153, LED154: KB_APTF1616V0, WallerLabLib:KB_RGBLED_APTF1616
- LED00, LED01, LED02, LED03, LED04, LED05, LED06, LED07, LED08, LED09, LED10, LED100, LED101, LED102, LED103, LED104, LED105, LED106, LED107, LED108, LED109, LED11, LED110, LED12, LED13, LED14, LED15, LED16, LED17, LED18, LED19, LED20, LED21, LED22, LED23, LED24, LED25, LED26, LED27, LED28, LED29, LED30, LED31, LED32, LED33, LED34, LED35, LED36, LED37, LED38, LED39, LED40, LED41, LED42, LED43, LED44, LED45, LED46, LED47, LED48, LED49, LED50, LED51, LED52, LED53, LED54, LED55, LED56, LED57, LED58, LED59, LED60, LED61, LED62, LED63, LED64, LED65, LED66, LED67, LED68, LED69, LED70, LED71, LED72, LED73, LED74, LED75, LED76, LED77, LED78, LED79, LED80, LED81, LED82, LED83, LED84, LED85, LED86, LED87, LED88, LED89, LED90, LED91, LED92, LED93, LED94, LED95, LED96, LED97, LED98, LED99: device ZacksLib:KB_RGBLED_APTF1616 -> WallerLabLib:KB_RGBLED_APTF1616
- moved LED108 272.1 mm to (-218.8, -17.1), turned to 0 degrees
- moved LED109 269.9 mm to (-220.7, -17.1), turned to 0 degrees
- moved LED101 264.9 mm to (-205.5, -16.8), turned to 0 degrees
- moved LED102 262.7 mm to (-207.4, -16.8), turned to 0 degrees
- moved LED103 260.6 mm to (-209.3, -16.9), turned to 0 degrees
- moved LED105 258.2 mm to (-213.1, -16.9), turned to 0 degrees
- moved LED106 256.1 mm to (-215.0, -17.0), turned to 0 degrees
- moved LED110 255.4 mm to (-222.6, -17.2), turned to 0 degrees
- moved LED107 253.9 mm to (-216.9, -17.1), turned to 0 degrees
- moved LED95 247.6 mm to (-194.1, -16.4), turned to 0 degrees
- moved LED97 245.4 mm to (-197.9, -16.6), turned to 0 degrees
- moved LED89 244.3 mm to (-182.7, -16.1), turned to 0 degrees
- moved LED98 243.5 mm to (-199.8, -16.6), turned to 0 degrees
- moved LED104 243.0 mm to (-211.2, -16.9), turned to 0 degrees
- moved LED90 242.1 mm to (-184.6, -16.2), turned to 0 degrees
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Other:
- board outline removed
