File: PlanarArrayCellScope/ArrayF_v0zp.sch (EAGLE design)
At the start: 111 parts

Commit message: Updated Planar Array Designs
Parts:
- removed LED00, LED01, LED02, LED03, LED04, LED05, LED06, LED07, LED08, LED09, LED10, LED100, LED101, LED102, LED103, LED104, LED105, LED106, LED107, LED108, LED109, LED11, LED110, LED12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: KB_APTF1616V0, ZacksLib:KB_APTF1616V0
