File: PlanarArrayCellScope/ArrayC_v3zp.brd (EAGLE design)
At the start: 75 x 75 mm, 96 parts, among them T1 TLC5955V0, T2 TLC5955V0, T3 TLC5955V0, T4 TLC5955V0, T5 TLC5955V0

Commit message: Planar Array partial route
Parts:
- removed FLANGE3: 6PINS_LEDFLANGEV1, WallerLabLib:6PIN_PADS
- added FLANGE4: 6PINS_LEDFLANGEV1, WallerLabLib:6PIN_PADS
- moved ARDUINO 76.3 mm to (24.9, 1.65), turned to 0 degrees
- moved FLANGE1 43.7 mm to (25.7, 18.6), turned to 0 degrees
Connections:
- net GND: now also ARDUINO.1, FLANGE4.GND; no longer ARDUINO.6, FLANGE3.GND
- net GSCLK: now also ARDUINO.2, FLANGE4.GSCLK; no longer ARDUINO.1, FLANGE3.GSCLK
- net LAT: now also ARDUINO.4, FLANGE4.LAT; no longer ARDUINO.2, FLANGE3.LAT
- net N$365: now also ARDUINO.5; no longer ARDUINO.4
- net N$53: now also FLANGE4.SIN; no longer U$8.SIN
- net N$54: now also ARDUINO.6; no longer FLANGE3.SIN
- net N$55: now also FLANGE4.SOUT, U$8.SIN; no longer ARDUINO.5, FLANGE3.SOUT
- net SCLK: now also FLANGE4.CLK; no longer FLANGE3.CLK
Routing:
- net N$365: track 0.00 -> 53.3 mm
- net GSCLK: track 5.69 -> 18.3 mm
- net SCLK: track 0.00 -> 12.4 mm
- net LAT: track 0.00 -> 12.1 mm
- net 3.3V: track 406.0 -> 410.9 mm
- net GND: track 376.1 -> 376.3 mm, vias 8 -> 9
