File: PlanarArrayCellScope/ArrayC_v3zp.sch (EAGLE design)
At the start: 10 parts

Commit message: Updated Planar Array Designs
Parts:
- removed U$10: 2PIN_PWR0.1HEADER, WallerLabLib:2PIN_PWR0.1HEADER
- removed U$6: TLC5955V0, WallerLabLib:TLC5955V0
- removed U$9: 5_PINSV1, WallerLabLib:5_PINSV1
- added ARDUINO: 6_PINSV2, WallerLabLib:6_PINSV2
- added FLANGE1, FLANGE2, FLANGE3: 6PINS_LEDFLANGEV1, WallerLabLib:6PINS_LEDFLANGEV1
- added LED: 3_PINS_RGBV1, WallerLabLib:3_PINS_RGBV1
- added LED00, LED01, LED02, LED03, LED04, LED05, LED06, LED07, LED08, LED09, LED10, LED11, LED12, LED13, LED14, LED15, LED16, LED17, LED18, LED19, LED20, LED21, LED22, LED23, LED24, LED25, LED26, LED27, LED28, LED29, LED30, LED31, LED32, LED33, LED34, LED35, LED36, LED37, LED38, LED39, LED40, LED41, LED42, LED43, LED44, LED45, LED46, LED47, LED48, LED49, LED50, LED51, LED52, LED53, LED54, LED55, LED56, LED57, LED58, LED59, LED60, LED61, LED62, LED63, LED64, LED65, LED66, LED67, LED68, LED69, LED70, LED71, LED72, LED73, LED74, LED75, LED76, LED77, LED78, LED79, LED80: KB_APTF1616V0, WallerLabLib:KB_APTF1616V0
- added T1, T2, T5: TLC5955V0, WallerLabLib:TLC5955V0
- U$1, U$2, U$3, U$4: value TLC5955V0 -> 2_PINS_FLANGEPOWERV1; device WallerLabLib:TLC5955V0 -> WallerLabLib:2_PINS_FLANGEPOWERV1
- U$8: value TLC5955V0 -> 6PINS_LEDFLANGEV1; device WallerLabLib:TLC5955V0 -> WallerLabLib:6PINS_LEDFLANGEV1
- renumbered U$5 to T3, U$7 to T4
Connections:
- removed net N$236: U$6.R0
- removed net N$237: U$6.G0
- removed net N$238: U$6.B0
- removed net N$239: U$6.R1
- removed net N$240: U$6.G1
- removed net N$241: U$6.B1
- removed net N$242: U$6.R2
- removed net N$243: U$6.G2
- removed net N$244: U$6.B2
- removed net N$245: U$6.R3
- removed net N$246: U$6.G3
- removed net N$247: U$6.B3
- removed net N$248: U$6.R4
- removed net N$249: U$6.G4
- removed net N$250: U$6.B4
- removed net N$251: U$6.R5
- removed net N$252: U$6.G5
- removed net N$253: U$6.B5
- removed net N$254: U$6.R6
- removed net N$255: U$6.G6
- removed net N$256: U$6.B6
- removed net N$257: U$6.R7
- removed net N$258: U$6.G7
- removed net N$259: U$6.B7
- removed net N$260: U$6.B8
- removed net N$261: U$6.G8
- removed net N$262: U$6.R8
- removed net N$263: U$6.B9
- removed net N$264: U$6.G9
- removed net N$265: U$6.R9
- removed net N$266: U$6.B10
- removed net N$267: U$6.G10
- removed net N$268: U$6.R10
- removed net N$269: U$6.B11
- removed net N$270: U$6.G11
- removed net N$271: U$6.B12
- removed net N$272: U$6.G12
- removed net N$273: U$6.R12
- removed net N$274: U$6.B13
- removed net N$275: U$6.G13
- removed net N$276: U$6.R13
- removed net N$277: U$6.B14
- removed net N$278: U$6.G14
- removed net N$279: U$6.R14
- removed net N$280: U$6.B15
- removed net N$281: U$6.G15
- removed net N$282: U$6.R15
- removed net N$330: U$8.R0
- removed net N$331: U$8.G0
- removed net N$332: U$8.B0
- removed net N$333: U$8.R1
- removed net N$334: U$8.G1
- removed net N$335: U$8.B1
- removed net N$336: U$8.R2
- removed net N$337: U$8.G2
- removed net N$338: U$8.B2
- removed net N$339: U$8.R3
- removed net N$340: U$8.G3
- removed net N$341: U$8.B3
- removed net N$342: U$8.R4
- removed net N$343: U$8.G4
- removed net N$344: U$8.B4
- removed net N$345: U$8.R5
- removed net N$346: U$8.G5
- removed net N$347: U$8.B5
- removed net N$348: U$8.R6
- removed net N$349: U$8.G6
- removed net N$350: U$8.B6
- removed net N$351: U$8.R7
- removed net N$352: U$8.G7
- removed net N$353: U$8.B7
- removed net N$354: U$8.B8
- removed net N$355: U$8.G8
- removed net N$356: U$8.R8
- removed net N$358: U$2.SOUT, U$6.SIN
- removed net N$359: U$6.SOUT, U$8.SIN
- removed net N$366: U$8.SOUT, U$9.4
- removed net N$368: U$2.R11
- removed net N$371: U$6.R11
- removed net N$48: U$2.R0
- removed net N$56: U$2.B2
- removed net N$57: U$2.R3
- removed net N$58: U$2.G3
- removed net N$59: U$2.B3
- removed net N$60: U$2.R4
- removed net N$61: U$2.G4
- removed net N$62: U$2.B4
- removed net N$63: U$2.R5
- removed net N$64: U$2.G5
- removed net N$65: U$2.B5
- removed net N$66: U$2.R6
- removed net N$67: U$2.G6
- removed net N$68: U$2.B6
- removed net N$69: U$2.R7
- removed net N$70: U$2.G7
- removed net N$71: U$2.B7
- removed net N$72: U$2.B8
- removed net N$73: U$2.G8
- removed net N$74: U$2.R8
- removed net N$75: U$2.B9
- removed net N$76: U$2.G9
- removed net N$77: U$2.R9
- removed net N$78: U$2.B10
- removed net N$79: U$2.G10
- removed net N$80: U$2.R10
- removed net N$81: U$2.B11
- removed net N$82: U$2.G11
- removed net N$83: U$2.B12
- removed net N$84: U$2.G12
- removed net N$85: U$2.R12
- removed net N$86: U$2.B13
- removed net N$87: U$2.G13
- removed net N$88: U$2.R13
- removed net N$89: U$2.B14
- removed net N$90: U$2.G14
- removed net N$91: U$2.R14
- removed net N$92: U$2.B15
- removed net N$93: U$2.G15
- removed net N$94: U$2.R15
- new net N$374: LED00.VCC, LED04.VCC, LED05.VCC, LED06.VCC, LED07.VCC, LED08.VCC, LED09.VCC, LED13.VCC, LED14.VCC, LED18.VCC, LED22.VCC, LED27.VCC, LED28.VCC, LED36.VCC, LED37.VCC, LED38.VCC
- new net N$384: LED15.VCC, LED16.VCC, LED17.VCC, LED23.VCC, LED24.VCC, LED25.VCC, LED26.VCC, LED35.VCC, LED42.VCC, LED43.VCC, LED44.VCC, LED52.VCC, LED53.VCC, LED62.VCC, LED71.VCC, LED80.VCC
- net 3.3V: now also LED01.VCC, LED02.VCC, LED03.VCC, LED10.VCC, LED11.VCC, LED12.VCC, LED19.VCC, LED20.VCC, LED21.VCC, LED29.VCC, LED30.VCC, LED31.VCC, LED32.VCC, LED33.VCC, LED34.VCC, LED39.VCC, LED40.VCC, LED41.VCC, LED45.VCC, LED46.VCC, LED47.VCC, LED48.VCC, LED49.VCC, LED50.VCC, LED51.VCC, LED54.VCC, LED55.VCC, LED56.VCC, LED57.VCC, LED58.VCC, LED59.VCC, LED60.VCC, LED61.VCC, LED63.VCC, LED64.VCC, LED65.VCC, LED66.VCC, LED67.VCC, LED68.VCC, LED69.VCC, LED70.VCC, LED72.VCC, LED73.VCC, LED74.VCC, LED75.VCC, LED76.VCC, LED77.VCC, LED78.VCC, LED79.VCC, T1.VCC, T2.VCC, T5.VCC; no longer U$10.VCC, U$6.VCC, U$8.VCC
- net GND: now also ARDUINO.6, FLANGE1.GND, FLANGE2.GND, FLANGE3.GND, T1.GND, T1.GND2, T1.PAD, T2.GND, T2.GND2, T2.PAD, T5.GND, T5.GND2, T5.PAD; no longer U$1.GND2, U$1.PAD, U$10.GND, U$2.GND2, U$2.PAD, U$3.GND2, U$3.PAD, U$4.GND2, U$4.PAD, U$6.GND, U$6.GND2, U$6.PAD, U$8.GND2, U$8.PAD
- net GSCLK: now also ARDUINO.1, FLANGE1.GSCLK, FLANGE2.GSCLK, FLANGE3.GSCLK, T1.GSCLK, T2.GSCLK, T5.GSCLK; no longer U$1.GSCLK, U$2.GSCLK, U$3.GSCLK, U$4.GSCLK, U$6.GSCLK, U$9.1(SQ)
- net LAT: now also ARDUINO.2, FLANGE1.LAT, FLANGE2.LAT, FLANGE3.LAT, T1.LAT, T2.LAT, T5.LAT; no longer U$1.LAT, U$2.LAT, U$3.LAT, U$4.LAT, U$6.LAT, U$9.2
- net N$1: now also LED40.R-, T5.R4; no longer U$1.R0
- net N$10: now also LED31.R-, T5.R1; no longer U$1.R3
- net N$100: now also LED10.B-, T1.B0; no longer U$3.B1
- net N$101: now also LED19.R-, T1.R5; no longer U$3.R2
- net N$102: now also LED19.G-, T1.G5; no longer U$3.G2
- net N$103: now also LED19.B-, T1.B5; no longer U$3.B2
- net N$104: now also LED29.R-, T1.R1; no longer U$3.R3
- net N$105: now also LED29.G-, T1.G1; no longer U$3.G3
- net N$106: now also LED29.B-, T1.B1; no longer U$3.B3
- net N$107: now also LED20.R-, T1.R2; no longer U$3.R4
- net N$108: now also LED20.G-, T1.G2; no longer U$3.G4
- net N$109: now also LED20.B-, T1.B2; no longer U$3.B4
- net N$11: now also LED31.G-, T5.G1; no longer U$1.G3
- net N$110: now also LED11.R-, T1.R6; no longer U$3.R5
- net N$111: now also LED11.G-, T1.G6; no longer U$3.G5
- net N$112: now also LED11.B-, T1.B6; no longer U$3.B5
- net N$113: now also LED12.R-, T1.R3; no longer U$3.R6
- net N$114: now also LED12.G-, T1.G3; no longer U$3.G6
- net N$115: now also LED12.B-, T1.B3; no longer U$3.B6
- net N$116: now also LED03.R-, T1.R7; no longer U$3.R7
- net N$117: now also LED03.G-, T1.G7; no longer U$3.G7
- net N$118: now also LED03.B-, T1.B7; no longer U$3.B7
- net N$119: now also LED00.B-, T1.B8; no longer U$3.B8
- net N$12: now also LED31.B-, T5.B1; no longer U$1.B3
- net N$120: now also LED00.G-, T1.G8; no longer U$3.G8
- net N$121: now also LED00.R-, T1.R8; no longer U$3.R8
- net N$122: now also LED09.B-, T1.B12; no longer U$3.B9
- net N$123: now also LED09.G-, T1.G12; no longer U$3.G9
- net N$124: now also LED09.R-, T1.R12; no longer U$3.R9
- net N$125: now also LED18.B-, T1.B9; no longer U$3.B10
- net N$126: now also LED18.G-, T1.G9; no longer U$3.G10
- net N$127: now also LED18.R-, T1.R9; no longer U$3.R10
- net N$128: now also LED28.B-, T1.B13; no longer U$3.B11
- net N$129: now also LED28.G-, T1.G13; no longer U$3.G11
- net N$13: now also LED32.R-, T5.R2; no longer U$1.R4
- net N$130: now also LED38.B-, T1.B14; no longer U$3.B12
- net N$131: now also LED38.G-, T1.G14; no longer U$3.G12
- net N$132: now also LED38.R-, T1.R14; no longer U$3.R12
- net N$133: now also LED27.B-, T1.B10; no longer U$3.B13
- net N$134: now also LED27.G-, T1.G10; no longer U$3.G13
- net N$135: now also LED27.R-, T1.R10; no longer U$3.R13
- net N$136: now also LED37.B-, T1.B15; no longer U$3.B14
- net N$137: now also LED37.G-, T1.G15; no longer U$3.G14
- net N$138: now also LED37.R-, T1.R15; no longer U$3.R14
- net N$139: now also LED36.B-, T1.B11; no longer U$3.B15
- net N$14: now also LED32.G-, T5.G2; no longer U$1.G4
- net N$140: now also LED36.G-, T1.G11; no longer U$3.G15
- net N$141: now also LED36.R-, T1.R11; no longer U$3.R15
- net N$142: now also LED44.R-, T3.R4; no longer T3.R0
- net N$143: now also LED08.R-, T2.R4; no longer U$4.R0
- net N$144: now also LED08.G-, T2.G4; no longer U$4.G0
- net N$145: now also LED08.B-, T2.B4; no longer U$4.B0
- net N$146: now also LED07.R-, T2.R0; no longer U$4.R1
- net N$147: now also LED07.G-, T2.G0; no longer U$4.G1
- net N$148: now also LED07.B-, T2.B0; no longer U$4.B1
- net N$149: now also LED06.R-, T2.R5; no longer U$4.R2
- net N$15: now also LED32.B-, T5.B2; no longer U$1.B4
- net N$150: now also LED06.G-, T2.G5; no longer U$4.G2
- net N$151: now also LED06.B-, T2.B5; no longer U$4.B2
- net N$152: now also LED05.R-, T2.R1; no longer U$4.R3
- net N$153: now also LED05.G-, T2.G1; no longer U$4.G3
- net N$154: now also LED05.B-, T2.B1; no longer U$4.B3
- net N$155: now also LED14.R-, T2.R2; no longer U$4.R4
- net N$156: now also LED14.G-, T2.G2; no longer U$4.G4
- net N$157: now also LED14.B-, T2.B2; no longer U$4.B4
- net N$158: now also LED04.R-, T2.R6; no longer U$4.R5
- net N$159: now also LED04.G-, T2.G6; no longer U$4.G5
- net N$16: now also LED33.R-, T5.R6; no longer U$1.R5
- net N$160: now also LED04.B-, T2.B6; no longer U$4.B5
- net N$161: now also LED13.R-, T2.R3; no longer U$4.R6
- net N$162: now also LED13.G-, T2.G3; no longer U$4.G6
- net N$163: now also LED13.B-, T2.B3; no longer U$4.B6
- net N$164: now also LED22.R-, T2.R7; no longer U$4.R7
- net N$165: now also LED22.G-, T2.G7; no longer U$4.G7
- net N$166: now also LED22.B-, T2.B7; no longer U$4.B7
- net N$167: now also LED35.B-, T2.B8; no longer U$4.B8
- net N$168: now also LED35.G-, T2.G8; no longer U$4.G8
- net N$169: now also LED35.R-, T2.R8; no longer U$4.R8
- net N$17: now also LED33.G-, T5.G6; no longer U$1.G5
- net N$170: now also LED23.B-, T2.B12; no longer U$4.B9
- net N$171: now also LED23.G-, T2.G12; no longer U$4.G9
- net N$172: now also LED23.R-, T2.R12; no longer U$4.R9
- net N$173: now also LED24.B-, T2.B9; no longer U$4.B10
- net N$174: now also LED24.G-, T2.G9; no longer U$4.G10
- net N$175: now also LED24.R-, T2.R9; no longer U$4.R10
- net N$176: now also LED25.B-, T2.B13; no longer U$4.B11
- net N$177: now also LED25.G-, T2.G13; no longer U$4.G11
- net N$178: now also LED26.B-, T2.B14; no longer U$4.B12
- net N$179: now also LED26.G-, T2.G14; no longer U$4.G12
- net N$18: now also LED33.B-, T5.B6; no longer U$1.B5
- net N$180: now also LED26.R-, T2.R14; no longer U$4.R12
- net N$181: now also LED15.B-, T2.B10; no longer U$4.B13
- net N$182: now also LED15.G-, T2.G10; no longer U$4.G13
- net N$183: now also LED15.R-, T2.R10; no longer U$4.R13
- net N$184: now also LED16.B-, T2.B15; no longer U$4.B14
- net N$185: now also LED16.G-, T2.G15; no longer U$4.G14
- net N$186: now also LED16.R-, T2.R15; no longer U$4.R14
- net N$187: now also LED17.B-, T2.B11; no longer U$4.B15
- net N$188: now also LED17.G-, T2.G11; no longer U$4.G15
- net N$189: now also LED17.R-, T2.R11; no longer U$4.R15
- net N$19: now also LED34.R-, T5.R3; no longer U$1.R6
- net N$190: now also LED44.G-, T3.G4; no longer T3.G0
- net N$191: now also LED44.B-, T3.B4; no longer T3.B0
- net N$192: now also LED43.R-, T3.R0; no longer T3.R1
- net N$193: now also LED43.G-, T3.G0; no longer T3.G1
- net N$194: now also LED43.B-, T3.B0; no longer T3.B1
- net N$195: now also LED42.R-, T3.R5; no longer T3.R2
- net N$196: now also LED42.G-, T3.G5; no longer T3.G2
- net N$197: now also LED42.B-, T3.B5; no longer T3.B2
- net N$198: now also LED52.R-, T3.R1; no longer T3.R3
- net N$199: now also LED52.G-, T3.G1; no longer T3.G3
- net N$2: now also LED40.G-, T5.G4; no longer U$1.G0
- net N$20: now also LED34.G-, T5.G3; no longer U$1.G6
- net N$200: now also LED52.B-, T3.B1; no longer T3.B3
- net N$201: now also LED53.R-, T3.R2; no longer T3.R4
- net N$202: now also LED53.G-, T3.G2; no longer T3.G4
- net N$203: now also LED53.B-, T3.B2; no longer T3.B4
- net N$204: now also LED62.R-, T3.R6; no longer T3.R5
- net N$205: now also LED62.G-, T3.G6; no longer T3.G5
- net N$206: now also LED62.B-, T3.B6; no longer T3.B5
- net N$207: now also LED71.R-, T3.R3; no longer T3.R6
- net N$208: now also LED71.G-, T3.G3; no longer T3.G6
- net N$209: now also LED71.B-, T3.B3; no longer T3.B6
- net N$21: now also LED34.B-, T5.B3; no longer U$1.B6
- net N$210: now also LED80.R-
- net N$211: now also LED80.G-
- net N$212: now also LED80.B-
- net N$213: now also LED79.B-
- net N$214: now also LED79.G-
- net N$215: now also LED79.R-
- net N$216: now also LED70.B-, T3.B12; no longer T3.B9
- net N$217: now also LED70.G-, T3.G12; no longer T3.G9
- net N$218: now also LED70.R-, T3.R12; no longer T3.R9
- net N$219: now also LED61.B-, T3.B9; no longer T3.B10
- net N$22: now also LED49.R-, T5.R7; no longer U$1.R7
- net N$220: now also LED61.G-, T3.G9; no longer T3.G10
- net N$221: now also LED61.R-, T3.R9; no longer T3.R10
- net N$222: now also LED78.B-, T3.B13; no longer T3.B11
- net N$223: now also LED78.G-, T3.G13; no longer T3.G11
- net N$224: now also LED77.B-, T3.B14; no longer T3.B12
- net N$225: now also LED77.G-, T3.G14; no longer T3.G12
- net N$226: now also LED77.R-, T3.R14; no longer T3.R12
- net N$227: now also LED69.B-, T3.B10; no longer T3.B13
- net N$228: now also LED69.G-, T3.G10; no longer T3.G13
- net N$229: now also LED69.R-, T3.R10; no longer T3.R13
- net N$23: now also LED49.G-, T5.G7; no longer U$1.G7
- net N$230: now also LED76.B-, T3.B15; no longer T3.B14
- net N$231: now also LED76.G-, T3.G15; no longer T3.G14
- net N$232: now also LED76.R-, T3.R15; no longer T3.R14
- net N$233: now also LED67.B-, T3.B11; no longer T3.B15
- net N$234: now also LED67.G-, T3.G11; no longer T3.G15
- net N$235: now also LED67.R-, T3.R11; no longer T3.R15
- net N$24: now also LED49.B-, T5.B7; no longer U$1.B7
- net N$25: now also LED48.B-, T5.B8; no longer U$1.B8
- net N$26: now also LED48.G-, T5.G8; no longer U$1.G8
- net N$27: now also LED48.R-, T5.R8; no longer U$1.R8
- net N$28: now also LED58.B-, T5.B12; no longer U$1.B9
- net N$283: now also LED63.R-, T4.R4; no longer T4.R0
- net N$284: now also LED63.G-, T4.G4; no longer T4.G0
- net N$285: now also LED63.B-, T4.B4; no longer T4.B0
- net N$286: now also LED57.R-, T4.R0; no longer T4.R1
- net N$287: now also LED57.G-, T4.G0; no longer T4.G1
- net N$288: now also LED57.B-, T4.B0; no longer T4.B1
- net N$289: now also LED65.R-, T4.R5; no longer T4.R2
- net N$29: now also LED58.G-, T5.G12; no longer U$1.G9
- net N$290: now also LED65.G-, T4.G5; no longer T4.G2
- net N$291: now also LED65.B-, T4.B5; no longer T4.B2
- net N$292: now also LED56.R-, T4.R1; no longer T4.R3
- net N$293: now also LED56.G-, T4.G1; no longer T4.G3
- net N$294: now also LED56.B-, T4.B1; no longer T4.B3
- net N$295: now also LED64.R-, T4.R2; no longer T4.R4
- net N$296: now also LED64.G-, T4.G2; no longer T4.G4
- net N$297: now also LED64.B-, T4.B2; no longer T4.B4
- net N$298: now also LED55.R-, T4.R6; no longer T4.R5
- net N$299: now also LED55.G-, T4.G6; no longer T4.G5
- net N$3: now also LED40.B-, T5.B4; no longer U$1.B0
- net N$30: now also LED58.R-, T5.R12; no longer U$1.R9
- net N$300: now also LED55.B-, T4.B6; no longer T4.B5
- net N$301: now also LED54.R-, T4.R3; no longer T4.R6
- net N$302: now also LED54.G-, T4.G3; no longer T4.G6
- net N$303: now also LED54.B-, T4.B3; no longer T4.B6
- net N$304: now also LED45.R-
- net N$305: now also LED45.G-
- net N$306: now also LED45.B-
- net N$307: now also LED39.B-
- net N$308: now also LED39.G-
- net N$309: now also LED39.R-
- net N$31: now also LED68.B-, T5.B9; no longer U$1.B10
- net N$310: now also LED46.B-, T4.B12; no longer T4.B9
- net N$311: now also LED46.G-, T4.G12; no longer T4.G9
- net N$312: now also LED46.R-, T4.R12; no longer T4.R9
- net N$313: now also LED47.B-, T4.B9; no longer T4.B10
- net N$314: now also LED47.G-, T4.G9; no longer T4.G10
- net N$315: now also LED47.R-, T4.R9; no longer T4.R10
- net N$316: now also LED66.B-, T4.B13; no longer T4.B11
- net N$317: now also LED66.G-, T4.G13; no longer T4.G11
- net N$318: now also LED75.B-, T4.B14; no longer T4.B12
- net N$319: now also LED75.G-, T4.G14; no longer T4.G12
- net N$32: now also LED68.G-, T5.G9; no longer U$1.G10
- net N$320: now also LED75.R-, T4.R14; no longer T4.R12
- net N$321: now also LED74.B-, T4.B10; no longer T4.B13
- net N$322: now also LED74.G-, T4.G10; no longer T4.G13
- net N$323: now also LED74.R-, T4.R10; no longer T4.R13
- net N$324: now also LED73.B-, T4.B15; no longer T4.B14
- net N$325: now also LED73.G-, T4.G15; no longer T4.G14
- net N$326: now also LED73.R-, T4.R15; no longer T4.R14
- net N$327: now also LED72.B-, T4.B11; no longer T4.B15
- net N$328: now also LED72.G-, T4.G11; no longer T4.G15
- net N$329: now also LED72.R-, T4.R11; no longer T4.R15
- net N$33: now also LED68.R-, T5.R9; no longer U$1.R10
- net N$34: now also LED59.B-, T5.B13; no longer U$1.B11
- net N$35: now also LED59.G-, T5.G13; no longer U$1.G11
- net N$357: now also FLANGE1.SIN, T5.SOUT; no longer U$1.SOUT, U$2.SIN
- net N$36: now also LED50.B-, T5.B14; no longer U$1.B12
- net N$360: now also T5.SIN; no longer U$1.SIN
- net N$362: now also T2.SOUT; no longer U$4.SOUT
- net N$363: now also T1.SOUT, T2.SIN; no longer U$3.SOUT, U$4.SIN
- net N$364: now also LED66.R-, T4.R13; no longer T4.R11
- net N$365: now also ARDUINO.4, T1.SIN; no longer U$3.SIN, U$9.5
- net N$37: now also LED50.G-, T5.G14; no longer U$1.G12
- net N$370: now also LED59.R-, T5.R13; no longer U$1.R11
- net N$372: now also LED78.R-, T3.R13; no longer T3.R11
- net N$373: now also LED25.R-, T2.R13; no longer U$4.R11
- net N$375: now also LED28.R-, T1.R13; no longer U$3.R11
- net N$38: now also LED50.R-, T5.R14; no longer U$1.R12
- net N$39: now also LED41.B-, T5.B10; no longer U$1.B13
- net N$4: now also LED21.R-, T5.R0; no longer U$1.R1
- net N$40: now also LED41.G-, T5.G10; no longer U$1.G13
- net N$41: now also LED41.R-, T5.R10; no longer U$1.R13
- net N$42: now also LED60.R-, T5.B15; no longer U$1.B14
- net N$43: now also LED60.G-, T5.G15; no longer U$1.G14
- net N$44: now also LED60.B-, T5.R15; no longer U$1.R14
- net N$45: now also LED51.B-, T5.B11; no longer U$1.B15
- net N$46: now also LED51.G-, T5.G11; no longer U$1.G15
- net N$47: now also LED51.R-, T5.R11; no longer U$1.R15
- net N$49: now also LED.RED, LED02.R-; no longer U$2.G0
- net N$5: now also LED21.G-, T5.G0; no longer U$1.G1
- net N$50: now also LED.BLUE, LED02.B-; no longer U$2.B0
- net N$51: now also LED.GREEN, LED02.G-; no longer U$2.R1
- net N$52: now also FLANGE1.SOUT, FLANGE2.SIN; no longer U$2.G1
- net N$53: now also FLANGE2.SOUT, U$8.SIN; no longer U$2.B1
- net N$54: now also FLANGE3.SIN, U$8.SOUT; no longer U$2.R2
- net N$55: now also ARDUINO.5, FLANGE3.SOUT; no longer U$2.G2
- net N$6: now also LED21.B-, T5.B0; no longer U$1.B1
- net N$7: now also LED30.R-, T5.R5; no longer U$1.R2
- net N$8: now also LED30.G-, T5.G5; no longer U$1.G2
- net N$9: now also LED30.B-, T5.B5; no longer U$1.B2
- net N$95: now also LED01.R-, T1.R4; no longer U$3.R0
- net N$96: now also LED01.G-, T1.G4; no longer U$3.G0
- net N$97: now also LED01.B-, T1.B4; no longer U$3.B0
- net N$98: now also LED10.R-, T1.R0; no longer U$3.R1
- net N$99: now also LED10.G-, T1.G0; no longer U$3.G1
- net SCLK: now also ARDUINO.3, FLANGE1.CLK, FLANGE2.CLK, FLANGE3.CLK, T1.SCLK, T2.SCLK, T5.SCLK, U$8.CLK; no longer U$1.SCLK, U$2.SCLK, U$3.SCLK, U$4.SCLK, U$6.SCLK, U$8.SCLK, U$9.3
Other:
- note removed: "6"
- note removed: "7"
- note removed: "8"

Commit message: Planar Array partial route
Parts:
- removed FLANGE3: 6PINS_LEDFLANGEV1, WallerLabLib:6PINS_LEDFLANGEV1
- added FLANGE4: 6PINS_LEDFLANGEV1, WallerLabLib:6PINS_LEDFLANGEV1
Connections:
- net GND: now also ARDUINO.1, FLANGE4.GND; no longer ARDUINO.6, FLANGE3.GND
- net GSCLK: now also ARDUINO.2, FLANGE4.GSCLK; no longer ARDUINO.1, FLANGE3.GSCLK
- net LAT: now also ARDUINO.4, FLANGE4.LAT; no longer ARDUINO.2, FLANGE3.LAT
- net N$365: now also ARDUINO.5; no longer ARDUINO.4
- net N$53: now also FLANGE4.SIN; no longer U$8.SIN
- net N$54: now also ARDUINO.6; no longer FLANGE3.SIN
- net N$55: now also FLANGE4.SOUT, U$8.SIN; no longer ARDUINO.5, FLANGE3.SOUT
- net SCLK: now also FLANGE4.CLK; no longer FLANGE3.CLK
Other:
- moved on the sheet: U$8
