File: DomedArrayAZ100/domeLedPcb.brd (EAGLE design)
At the start: 172.8 x 247.8 mm, 117 parts

Commit message: new 4P X 8S device and updated DomedArray board
Parts:
- removed U$1: 2PIN_PWR4-8-16MM, WallerLabLib:2PIN_HOLES_PWR
- added BASE_CONNECTOR: 4POWER_8SIGNALMATING_BOARD, WallerLabLib:4POWER_8SIGNAL
Connections:
- net DATA_IN: now also BASE_CONNECTOR.B4_B, BASE_CONNECTOR.B4_T
- net DATA_OUT: now also BASE_CONNECTOR.B5_B, BASE_CONNECTOR.B5_T
- net GND: now also BASE_CONNECTOR.A3_B, BASE_CONNECTOR.A3_T, BASE_CONNECTOR.A4_B, BASE_CONNECTOR.A4_T; no longer U$1.P$1
- net GSCLK: now also BASE_CONNECTOR.B1_B, BASE_CONNECTOR.B1_T
- net LAT: now also BASE_CONNECTOR.B2_B, BASE_CONNECTOR.B2_T
- net SCLK: now also BASE_CONNECTOR.B3_B, BASE_CONNECTOR.B3_T
- net VCC: now also BASE_CONNECTOR.A1_B, BASE_CONNECTOR.A1_T, BASE_CONNECTOR.A2_B, BASE_CONNECTOR.A2_T; no longer U$1.P$2
Routing:
- net DATA_IN: track 13.8 -> 326.4 mm, vias 0 -> 1
- net LAT: track 445.1 -> 514.2 mm, vias 20 -> 21
- net GND: track 548.3 -> 582.6 mm, vias 14 -> 15
- net VCC: track 1179.5 -> 1210.0 mm, vias 18 -> 19
- net SCLK: track 408.8 -> 438.9 mm, vias 5 -> 7
- net GSCLK: track 347.2 -> 374.9 mm, vias 11 -> 12
- net DATA_OUT: track 261.1 -> 281.4 mm, vias 2 -> 3
Other:
- board size 172.8 x 247.8 mm -> 172.8 x 240.2 mm

Commit message: Updated Dome PCB layout dimensions
Routing:
- net VCC: track 1210.0 -> 1195.9 mm
- net N$63: track 26.0 -> 25.3 mm
Other:
- board size 172.8 x 240.2 mm -> 177 x 247.5 mm
- board text added: "BD-Slice_r2.0"
- board text removed: "BD-Slice_r1.0"
